File: PCB/hackpad.kicad_pcb (KiCad board)
At the start: 2 copper layers, 63.2 x 81 mm, 7 parts, among them SW1 SW_Push, SW2 SW_Push, SW3 SW_Push, SW4 SW_Push, U1 XIAO-RP2040-DIP

Commit message: updated to be submitable
Parts:
- added SW5: SW_Push, Button_Switch_Keyboard:SW_Cherry_MX_1.00u_PCB, F.Cu at (81.2, 114.0)
- moved D2 20.2 mm to (81.2, 105.1)
Connections:
- U1 pad 3: unconnected-(U1-GPIO28/ADC2/A2-Pad3) -> Net-(U1-GPIO28/ADC2/A2)
Routing:
- net GND: track 199.0 -> 0.00 mm
- net +5V: track 107.9 -> 0.00 mm
- net Net-(U1-GPIO3/MOSI): track 82.8 -> 0.00 mm
- net Net-(D1-DOUT): track 76.2 -> 0.00 mm
- net Net-(U1-GPIO4/MISO): track 58.0 -> 0.00 mm
- net Net-(U1-GPIO2/SCK): track 47.8 -> 1.50 mm
- net Net-(U1-GPIO1/RX): track 37.4 -> 0.91 mm
- net Net-(D1-DIN): track 35.7 -> 0.00 mm
Other:
- board text added: "its in the shape of an l because of all of the ls i took making this"
